File: Autonomous_Rover.kicad_pcb (KiCad board)
At the start: 2 copper layers, 112 x 65 mm, 40 parts, among them M2_1 MountingHole_Pad, M2_2 MountingHole_Pad, M2_3 MountingHole_Pad, Q1 AO3400A, Q2 AO3400A

Commit message: Reduction in size
Move the components around to save some space
Parts:
- removed PPTC1: Polyfuse, Fuse:Fuse_1812_4532Metric
- added F1: 2.0A Hold / 3.5A Trip (16V+), Fuse:Fuse_2920_7451Metric, F.Cu at (188.6, 123.2)
- C7: renamed from C10UF1; value 10 micro F -> 10uF
- C8: renamed from C10UF2; value 10 Micro F -> 10uF
- H1: renamed from M2_1; value MountingHole_Pad -> M2
- H2: renamed from M2_2; value MountingHole_Pad -> M2
- H3: renamed from M2_3; value MountingHole_Pad -> M2
- J1: renamed from VL53L5X_R1; value VL53L5X_RIGHT -> VL53L5X_R
- J10: renamed from ESP32_L1; value ESP32_LEFT -> ESP32_L
- J11: renamed from ESP32_R1; value ESP32_RIGHT -> ESP32_R
- J12: renamed from 5V1; value 5V Socket -> 5V
- J14: renamed from POWER1; value Power Input -> POWER
- J3: renamed from VL53L5X_L1; value VL53L5X_LEFT -> VL53L5X_L
- J4: renamed from HC-SR04_M1; value HC-SR04_MID -> HC-SR04_M
- J5: renamed from VL53L5X_M1; value VL53L5X_MID -> VL53L5X_M
- J6: renamed from 3V3; value 3V Socket -> 3V
- J9: renamed from UART1; value EXTRA GPIO -> UART
- R1: renamed from R10K1; value ~ -> 10k
- moved J15 29.2 mm to (185.8, 72.4), turned to 180 degrees
- moved J6 27.7 mm to (153.2, 74.9)
- moved J13 27.7 mm to (153.2, 83.6)
- moved Q1 21.7 mm to (178.4, 78.1)
- moved R2 20.5 mm to (178.1, 80.8), turned to 180 degrees
- moved R1 16.6 mm to (175.3, 81.0), turned to 90 degrees
- moved J12 14.1 mm to (185.8, 76.1)
- moved D1 7.22 mm to (185.4, 94.5), turned to -90 degrees
- moved J8 6.44 mm to (185.8, 84.8)
- moved C8 6.35 mm to (163.7, 72.1), turned to -90 degrees
- moved BZ1 6.32 mm to (194.2, 102.7)
- moved C7 6.14 mm to (172.8, 72.3), turned to -90 degrees
- moved J14 5.66 mm to (190.9, 117.2), turned to 90 degrees
- moved J16 4.42 mm to (191.5, 71.0)
- moved R7 3.24 mm to (178.1, 113.7), turned to 180 degrees
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- renumbered BUZZER1 to BZ1, C100NF1 to C1, C100NF2 to C2, C100NF3 to C3, C100NF4 to C4, C100NF5 to C5, C100NF6 to C6, GND2 to J13, LIGHT1 to J15, MOTOR1 to J16, VEML7700 to J2, BNO085 to J7, GND1 to J8, R101 to R2, R1K1 to R3, R1K2 to R4, R10K2 to R5, R10K3 to R6, R102 to R7, 3V3OUT1 to U1
Routing:
- net SCL: track 149.3 -> 180.4 mm
- net GND: track 21.4 -> 2.54 mm, vias 20 -> 35
- net +3V3: track 256.9 -> 240.4 mm, vias 1 -> 0
- net +5V: track 157.2 -> 147.2 mm
- net SDA: track 146.2 -> 155.2 mm
- net /LPN_M: track 59.3 -> 52.5 mm
- net Net-(J14-Pin_1): track 12.3 -> 6.45 mm
- net /UART0_RX: track 34.8 -> 40.0 mm
- net Net-(J15-Pin_1): track 14.9 -> 10.0 mm
- net /R_IS: track 19.6 -> 15.5 mm
- net /BUZZ: track 7.08 -> 3.45 mm
- net /L_IS: track 19.3 -> 15.7 mm
- net /L_RPWM: track 13.5 -> 9.96 mm
- net /L_LPWM: track 13.5 -> 9.98 mm
- net /R_RPWM: track 13.5 -> 9.99 mm
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Other:
- board size 112 x 65 mm -> 109.5 x 65 mm
- board text added: "+"
- board text added: "-"
- board text added: "ESP32-S3-DEVKITC-1"
- board text added: "USB"
- board text added: "^"
