File: Autonomous_Rover.kicad_sch (KiCad schematic)
At the start: 40 parts, among them M2_1 MountingHole_Pad, M2_2 MountingHole_Pad, M2_3 MountingHole_Pad, Q1 AO3400A, Q2 AO3400A

Commit message: Reduction in size
Move the components around to save some space
Parts:
- C7: renamed from C10UF1; value 10 micro F -> 10uF
- C8: renamed from C10UF2; value 10 Micro F -> 10uF
- F1: renamed from PPTC1; value Polyfuse -> 2.0A Hold / 3.5A Trip (16V+); footprint Fuse:Fuse_1812_4532Metric -> Fuse:Fuse_2920_7451Metric
- H1: renamed from M2_1; value MountingHole_Pad -> M2
- H2: renamed from M2_2; value MountingHole_Pad -> M2
- H3: renamed from M2_3; value MountingHole_Pad -> M2
- J1: renamed from VL53L5X_R1; value VL53L5X_RIGHT -> VL53L5X_R
- J10: renamed from ESP32_L1; value ESP32_LEFT -> ESP32_L
- J11: renamed from ESP32_R1; value ESP32_RIGHT -> ESP32_R
- J12: renamed from 5V1; value 5V Socket -> 5V
- J14: renamed from POWER1; value Power Input -> POWER
- J3: renamed from VL53L5X_L1; value VL53L5X_LEFT -> VL53L5X_L
- J4: renamed from HC-SR04_M1; value HC-SR04_MID -> HC-SR04_M
- J5: renamed from VL53L5X_M1; value VL53L5X_MID -> VL53L5X_M
- J6: renamed from 3V3; value 3V Socket -> 3V
- J9: renamed from UART1; value EXTRA GPIO -> UART
- R1: renamed from R10K1; value (none) -> 10k
- renumbered BUZZER1 to BZ1, C100NF1 to C1, C100NF2 to C2, C100NF3 to C3, C100NF4 to C4, C100NF5 to C5, C100NF6 to C6, GND2 to J13, LIGHT1 to J15, MOTOR1 to J16, VEML7700 to J2, BNO085 to J7, GND1 to J8, R101 to R2, R1K1 to R3, R1K2 to R4, R10K2 to R5, R10K3 to R6, R102 to R7, 3V3OUT1 to U1
Other:
- moved on the sheet: C8
